File: espduino.sch (KiCad schematic (older format))
At the start: 17 parts, among them CON101 USB-MICRO-B, CON102 AVR-ISP-6, IC101 ATMEGA328-P, P101 CONN_01X12, P102 CONN_01X12, P103 FTDI, P104 CONN_01X02, P105 CONN_01X03, SW101 SPST, X101 16Mhz

Commit message: Version 0.2
Parts:
- removed IC101: ATMEGA328-P, TQFP32, symbol ATMEGA328-P
- added IC101: ATMEGA328P-A, footprints:TQFP32_08, symbol ATMEGA328P-A
- C101, C102, C103, C104: symbol C -> C-RESCUE-espduino
- CON101: footprint (none) -> footprints:USB_Micro-B
- CON102: footprint AVR-ISP-6 -> Pin_Headers:Pin_Header_Straight_2x03; symbol AVR-ISP-6 -> AVR-ISP-6-RESCUE-espduino
- D101: symbol LED -> LED-RESCUE-espduino
- P101: renamed from P105; footprint (none) -> Pin_Headers:Pin_Header_Straight_1x03
- P102: renamed from P101; footprint Pin_Headers:Pin_Header_Straight_1x06 -> Pin_Headers:Pin_Header_Straight_1x12
- P104: renamed from P103; footprint Pin_Headers:Pin_Header_Straight_1x12 -> Pin_Headers:Pin_Header_Angled_1x06
- P105: renamed from P104; footprint (none) -> Pin_Headers:Pin_Header_Straight_1x02
- R101, R102: symbol R -> R-RESCUE-espduino
- SW101: footprint LittlebushLogicFootPrints:4x4_Tactile_SMD_switch -> footprints:4x4_Tactile_SMD_switch
- renumbered P102 to P103
Other:
- moved on the sheet: CON102
Changed lines of the file:
@@
 EESchema Schematic File Version 2
+LIBS:espduino-rescue
 LIBS:power
 LIBS:device
@@
 LIBS:memory
 LIBS:xilinx
-LIBS:special
 LIBS:microcontrollers
 LIBS:dsp
@@
 LIBS:valves
 LIBS:littlebush
+LIBS:ab2_7segment
+LIBS:ab2_audio
+LIBS:ab2_buffer
+LIBS:ab2_capacitor
+LIBS:ab2_connectivity
+LIBS:ab2_dac
+LIBS:ab2_diode
+LIBS:ab2_gpio_expansion
+LIBS:ab2_header
+LIBS:ab2_idc
+LIBS:ab2_inductor
+LIBS:ab2_input_devices
+LIBS:ab2_jumper
+LIBS:ab2_lcd
+LIBS:ab2_led
+LIBS:ab2_opamp
+LIBS:ab2_pot
+LIBS:ab2_power
+LIBS:ab2_regulator
+LIBS:ab2_relay
+LIBS:ab2_resistor
+LIBS:ab2_sensor
+LIBS:ab2_stepper
+LIBS:ab2_supply
+LIBS:ab2_terminal_block
+LIBS:ab2_test
+LIBS:ab2_transistor
+LIBS:ab2_uC
+LIBS:ab2_usb
+LIBS:ab2_xtal
 LIBS:espduino-cache
 EELAYER 25 0
@@
 $Descr A4 11693 8268
 encoding utf-8
-Sheet 1 5
+Sheet 1 6
 Title ""
 Date ""
@@
 $EndDescr
 $Comp
-L CONN_01X06 P103
+L CONN_01X06 P104
 U 1 1 54EEFCA8
 P 7300 2850
-F 0 "P103" H 7300 3200 50  0000 C CNN
+F 0 "P104" H 7300 3200 50  0000 C CNN
 F 1 "FTDI" V 7400 2850 50  0000 C CNN
-F 2 "Pin_Headers:Pin_Header_Straight_1x12" H 7300 2850 60  0001 C CNN
+F 2 "Pin_Headers:Pin_Header_Angled_1x06" H 7300 2850 60  0001 C CNN
 F 3 "" H 7300 2850 60  0000 C CNN
 	1    7300 2850
@@
 DTR
 $Comp
-L CONN_01X12 P101
+L CONN_01X12 P102
 U 1 1 54EEFCBA
 P 5650 3150
-F 0 "P101" H 5650 3800 50  0000 C CNN
+F 0 "P102" H 5650 3800 50  0000 C CNN
 F 1 "CONN_01X12" V 5750 3150 50  0000 C CNN
-F 2 "Pin_Headers:Pin_Header_Straight_1x06" H 5650 3150 60  0001 C CNN
+F 2 "Pin_Headers:Pin_Header_Straight_1x12" H 5650 3150 60  0001 C CNN
 F 3 "" H 5650 3150 60  0000 C CNN
 	1    5650 3150
@@
 $EndComp
 $Comp
-L CONN_01X12 P102
+L CONN_01X12 P103
 U 1 1 54EEFCBB
 P 6900 3150
-F 0 "P102" H 6900 3800 50  0000 C CNN
+F 0 "P103" H 6900 3800 50  0000 C CNN
 F 1 "CONN_01X12" V 7000 3150 50  0000 C CNN
 F 2 "Pin_Headers:Pin_Header_Straight_1x12" H 6900 3150 60  0001 C CNN
@@
 $EndComp
 $Comp
-L VCC #PWR104
+L VCC #PWR01
 U 1 1 54F43D94
 P 1550 4650
-F 0 "#PWR104" H 1550 4500 60  0001 C CNN
+F 0 "#PWR01" H 1550 4500 60  0001 C CNN
 F 1 "VCC" H 1550 4800 60  0000 C CNN
 F 2 "" H 1550 4650 60  0000 C CNN
@@
 $EndComp
 $Comp
-L C C101
+L C-RESCUE-espduino C101
 U 1 1 54F43EE2
 P 1350 5550
@@
 $EndComp
 $Comp
-L GND #PWR101
+L GND #PWR02
 U 1 1 54F43FD7
 P 1350 5750
-F 0 "#PWR101" H 1350 5500 60  0001 C CNN
+F 0 "#PWR02" H 1350 5500 60  0001 C CNN
 F 1 "GND" H 1350 5600 60  0000 C CNN
 F 2 "" H 1350 5750 60  0000 C CNN
@@
 $EndComp
 $Comp
-L GND #PWR105
+L GND #PWR03
 U 1 1 54F442ED
 P 1650 7050
-F 0 "#PWR105" H 1650 6800 60  0001 C CNN
+F 0 "#PWR03" H 1650 6800 60  0001 C CNN
 F 1 "GND" H 1650 6900 60  0000 C CNN
 F 2 "" H 1650 7050 60  0000 C CNN
@@
 $EndComp
 $Comp
-L C C102
+L C-RESCUE-espduino C102
 U 1 1 54F4538D
 P 5050 5100
@@
 $EndComp
 $Comp
-L C C103
+L C-RESCUE-espduino C103
 U 1 1 54F453F0
 P 5050 5700
@@
 Connection ~ 4700 5700
 $Comp
-L GND #PWR109
+L GND #PWR04
 U 1 1 54F456F6
 P 5350 5100
-F 0 "#PWR109" H 5350 4850 60  0001 C CNN
+F 0 "#PWR04" H 5350 4850 60  0001 C CNN
 F 1 "GND" H 5350 4950 60  0000 C CNN
 F 2 "" H 5350 5100 60  0000 C CNN
@@
 $EndComp
 $Comp
-L GND #PWR110
+L GND #PWR05
 U 1 1 54F45748
 P 5350 5700
-F 0 "#PWR110" H 5350 5450 60  0001 C CNN
+F 0 "#PWR05" H 5350 5450 60  0001 C CNN
 F 1 "GND" H 5350 5550 60  0000 C CNN
 F 2 "" H 5350 5700 60  0000 C CNN
@@
 D7
 $Comp
-L R R102
+L R-RESCUE-espduino R102
 U 1 1 54F46AF4
 P 4700 6350
@@
 F 0 "SW101" H 5200 6900 50  0000 C CNN
 F 1 "SPST" H 5200 6700 50  0000 C CNN
-F 2 "LittlebushLogicFootPrints:4x4_Tactile_SMD_switch" H 5200 6800 60  0001 C CNN
+F 2 "footprints:4x4_Tactile_SMD_switch" H 5200 6800 60  0001 C CNN
 F 3 "" H 5200 6800 60  0000 C CNN
 	1    5200 6800
@@
 	4500 6600 5000 6600
 $Comp
-L VCC #PWR108
+L VCC #PWR06
 U 1 1 54F46FC5
 P 4700 6100
-F 0 "#PWR108" H 4700 5950 60  0001 C CNN
+F 0 "#PWR06" H 4700 5950 60  0001 C CNN
 F 1 "VCC" H 4700 6250 60  0000 C CNN
 F 2 "" H 4700 6100 60  0000 C CNN
@@
 $EndComp
 $Comp
-L C C104
+L C-RESCUE-espduino C104
 U 1 1 54F4724A
 P 5200 6350
@@
 	4250 4800 4400 4800
 $Comp
-L LED D101
+L LED-RESCUE-espduino D101
 U 1 1 54F47743
 P 5100 4800
@@
 $EndComp
 $Comp
-L R R101
+L R-RESCUE-espduino R101
 U 1 1 54F47873
 P 4650 4800
@@
 D10
 $Comp
-L CONN_01X02 P104
+L CONN_01X02 P105
 U 1 1 54F6EBD0
 P 7300 3500
-F 0 "P104" H 7300 3650 50  0000 C CNN
+F 0 "P105" H 7300 3650 50  0000 C CNN
 F 1 "CONN_01X02" V 7450 3500 50  0000 C CNN
-F 2 "" H 7300 3500 60  0000 C CNN
+F 2 "Pin_Headers:Pin_Header_Straight_1x02" H 7300 3500 60  0001 C CNN
 F 3 "" H 7300 3500 60  0000 C CNN
 	1    7300 3500
@@
 Connection ~ 5700 6800
 $Comp
-L GND #PWR112
+L GND #PWR07
 U 1 1 54F71020
 P 5950 6800
-F 0 "#PWR112" H 5950 6550 60  0001 C CNN
+F 0 "#PWR07" H 5950 6550 60  0001 C CNN
 F 1 "GND" H 5950 6650 60  0000 C CNN
 F 2 "" H 5950 6800 60  0000 C CNN
@@
 	5700 6800 5950 6800
 $Comp
-L GND #PWR111
+L GND #PWR08
 U 1 1 54F713D5
 P 5650 4800
-F 0 "#PWR111" H 5650 4550 60  0001 C CNN
+F 0 "#PWR08" H 5650 4550 60  0001 C CNN
 F 1 "GND" H 5650 4650 60  0000 C CNN
 F 2 "" H 5650 4800 60  0000 C CNN
@@
 $EndComp
 $Comp
-L PWR_FLAG #FLG101
+L PWR_FLAG #FLG09
 U 1 1 54F71E44
 P 5950 6800
-F 0 "#FLG101" H 5950 6895 30  0001 C CNN
+F 0 "#FLG09" H 5950 6895 30  0001 C CNN
 F 1 "PWR_FLAG" H 5950 6980 30  0000 C CNN
 F 2 "" H 5950 6800 60  0000 C CNN
@@
 	1500 3100 1850 3100
 $Comp
-L GND #PWR103
+L GND #PWR010
 U 1 1 5538D63B
 P 1500 3650
-F 0 "#PWR103" H 1500 3400 60  0001 C CNN
+F 0 "#PWR010" H 1500 3400 60  0001 C CNN
 F 1 "GND" H 1500 3500 60  0000 C CNN
 F 2 "" H 1500 3650 60  0000 C CNN
@@
 	2300 1325 2700 1325
 $Comp
-L CONN_01X03 P105
+L CONN_01X03 P101
 U 1 1 559105BB
 P 2300 2200
-F 0 "P105" H 2300 2400 50  0000 C CNN
+F 0 "P101" H 2300 2400 50  0000 C CNN
 F 1 "CONN_01X03" V 2400 2200 50  0000 C CNN
-F 2 "" H 2300 2200 60  0000 C CNN
+F 2 "Pin_Headers:Pin_Header_Straight_1x03" H 2300 2200 60  0001 C CNN
 F 3 "" H 2300 2200 60  0000 C CNN
 	1    2300 2200
@@
 $EndComp
 $Comp
-L GND #PWR107
+L GND #PWR011
 U 1 1 559107D6
 P 2725 2150
-F 0 "#PWR107" H 2725 1900 60  0001 C CNN
+F 0 "#PWR011" H 2725 1900 60  0001 C CNN
 F 1 "GND" H 2725 2000 60  0000 C CNN
 F 2 "" H 2725 2150 60  0000 C CNN
@@
 $EndComp
 $Comp
-L VCC #PWR106
+L VCC #PWR012
 U 1 1 5591085F
 P 1900 2175
-F 0 "#PWR106" H 1900 2025 60  0001 C CNN
+F 0 "#PWR012" H 1900 2025 60  0001 C CNN
 F 1 "VCC" H 1900 2325 60  0000 C CNN
 F 2 "" H 1900 2175 60  0000 C CNN
@@
 	1900 2000 1900 2175
 $Comp
-L +5V #PWR102
+L +5V #PWR013
 U 1 1 55911357
 P 1500 3100
-F 0 "#PWR102" H 1500 2950 60  0001 C CNN
+F 0 "#PWR013" H 1500 2950 60  0001 C CNN
 F 1 "+5V" H 1500 3240 60  0000 C CNN
 F 2 "" H 1500 3100 60  0000 C CNN
@@
 F 0 "CON101" H 2050 3650 50  0000 C CNN
 F 1 "USB-MICRO-B" H 2200 2950 50  0000 C CNN
-F 2 "" H 2350 3200 50  0000 C CNN
+F 2 "footprints:USB_Micro-B" H 2350 3200 50  0001 C CNN
 F 3 "" H 2350 3200 50  0000 C CNN
 	1    2350 3300
@@
 Wire Wire Line
 	3025 3100 2850 3100
-$Comp
-L ATMEGA328-P IC101
-U 1 1 5593AEC4
-P 2650 5850
-F 0 "IC101" H 1900 7100 40  0000 L BNN
-F 1 "ATMEGA328-P" H 3050 4450 40  0000 L BNN
-F 2 "TQFP32" H 2650 5850 30  0000 C CIN
-F 3 "" H 2650 5850 60  0000 C CNN
-	1    2650 5850
-	1    0    0    -1
-$EndComp
 Wire Wire Line
 	1650 6950 1650 7050
 $Sheet
-S 9725 1100 825  550
+S 10325 600  825  550
 U 559CE2A1
 F0 "Freezy" 60
@@
 $EndSheet
 $Comp
-L AVR-ISP-6 CON102
+L AVR-ISP-6-RESCUE-espduino CON102
 U 1 1 559DF1DC
 P 7575 4500
 F 0 "CON102" H 7495 4740 50  0000 C CNN
 F 1 "AVR-ISP-6" H 7335 4270 50  0000 L BNN
-F 2 "AVR-ISP-6" V 7055 4540 50  0001 C CNN
+F 2 "Pin_Headers:Pin_Header_Straight_2x03" V 7055 4540 50  0001 C CNN
 F 3 "" H 7575 4500 60  0000 C CNN
 	1    7575 4500
@@
 Text Label 7000 4600 2    60   ~ 0
 RESET
+$Sheet
+S 9850 1950 1000 1050
+U 55A4DB37
+F0 "Charger" 60
+F1 "charger.sch" 60
+$EndSheet
+$Comp
+L ATMEGA328P-A IC101
+U 1 1 55A61801
+P 2650 5850
+F 0 "IC101" H 1900 7100 40  0000 L BNN
+F 1 "ATMEGA328P-A" H 3050 4450 40  0000 L BNN
+F 2 "footprints:TQFP32_08" H 2650 5850 30  0000 C CIN
+F 3 "" H 2650 5850 60  0000 C CNN
+	1    2650 5850
+	1    0    0    -1
+$EndComp
 $EndSCHEMATC
